File: kicad_source/SonarExtenderI2C.sch (KiCad schematic (older format))
At the start: 32 parts

Commit message: added auto measure circuit and echo status
Parts:
- added U?: 74xx4002, symbol IC_logic:74xx4002
- U: symbol IC_logic:NE555 -> SonarExtenderI2C-rescue:NE555-IC_logic
- U? (x4): symbol IC_logic:74xx590 -> SonarExtenderI2C-rescue:74xx590-IC_logic
- U?: symbol IC_logic:74xx175 -> SonarExtenderI2C-rescue:74xx175-IC_logic
- U?: symbol IC_logic:74xx04 -> SonarExtenderI2C-rescue:74xx04-IC_logic
- U?: symbol IC_logic:74xx138 -> SonarExtenderI2C-rescue:74xx138-IC_logic
Connections:
- net labels added: AUTO
- wire segments 299 -> 309
- no-connect marks 16 -> 20
Other:
- moved on the sheet: C?
