File: kicad_source/SonarExtenderI2C.sch (KiCad schematic (older format))
At the start: 33 parts

Commit message: changed and colorized logic table
Connections:
- net labels added: T0, T1, T2, T3
- wire segments 309 -> 313
Changed lines of the file:
@@
 Text Label 3200 3800 0    50   ~ 0
 STATUS_ECHO
-Text Label 3200 3900 0    50   ~ 0
-EN0
-Text Label 3200 4000 0    50   ~ 0
-EN1
-Text Label 3200 4100 0    50   ~ 0
-EN2
-Text Label 3200 4200 0    50   ~ 0
-EN3
 $Comp
 L mechanical-connectors:CONN_01X04 P?
@@
 	5600 4600 5000 4600
 Wire Wire Line
-	5600 4400 5000 4400
-Wire Wire Line
 	5600 4200 5000 4200
 Wire Wire Line
 	5600 4000 5000 4000
 Wire Wire Line
-	3100 3900 4300 3900
-Wire Wire Line
 	4300 4100 4200 4100
 Wire Wire Line
 	4200 4100 4200 4000
 Wire Wire Line
-	3100 4000 4200 4000
-Wire Wire Line
 	4100 4300 4100 4100
 Wire Wire Line
-	3100 4100 4100 4100
-Wire Wire Line
 	4100 4300 4300 4300
 Wire Wire Line
@@
 Wire Wire Line
 	3950 4500 3950 4200
-Wire Wire Line
-	3100 4200 3950 4200
 Wire Wire Line
 	5300 3900 5600 3900
@@
 Text Label 4200 3450 0    50   ~ 0
 CLK_10KHZ
-Text Label 5350 3900 0    50   ~ 0
-EN0
-Text Label 5350 4100 0    50   ~ 0
-EN1
-Text Label 5350 4300 0    50   ~ 0
-EN2
-Text Label 5350 4500 0    50   ~ 0
-EN3
 $Comp
 L power-supply:+3V3 #PWR?
@@
 Text GLabel 7300 6150 0    50   Input ~ 0
 CNT3
+Wire Wire Line
+	4300 3900 3850 3900
+Wire Wire Line
+	4200 4000 3850 4000
+Wire Wire Line
+	4100 4100 3850 4100
+Wire Wire Line
+	3950 4200 3850 4200
+Text GLabel 3850 3900 0    50   Input ~ 0
+EN0
+Text GLabel 3850 4000 0    50   Input ~ 0
+EN1
+Text GLabel 3850 4100 0    50   Input ~ 0
+EN2
+Text GLabel 3850 4200 0    50   Input ~ 0
+EN3
+Wire Wire Line
+	5600 4400 5000 4400
+Wire Wire Line
+	3100 3900 3400 3900
+Wire Wire Line
+	3100 4000 3400 4000
+Wire Wire Line
+	3100 4100 3400 4100
+Wire Wire Line
+	3100 4200 3400 4200
+Text GLabel 3400 3900 2    50   Output ~ 0
+T0
+Text GLabel 3400 4000 2    50   Output ~ 0
+T1
+Text GLabel 3400 4100 2    50   Output ~ 0
+T2
+Text GLabel 3400 4200 2    50   Output ~ 0
+T3
 $EndSCHEMATC

Commit message: added connector for I2C, annotated schematic
Parts:
- added CN1: CONN_01X05, symbol mechanical-connectors:CONN_01X05
- added CN2: CONN_01X04, symbol mechanical-connectors:CONN_01X04
- gave numbers to parts that had none: 32
- renumbered U to U1
Connections:
- net labels added: I2C_INT
- wire segments 313 -> 326
Other:
- note added: "Qwiic connector"

Commit message: exchanged I2C expanders to TCA9535 (16 bit type), generated schematic pdf
Parts:
- removed C2: 100nF, capacitors:C_0603, symbol devices:C_0603
- removed U2, U3: TCA9534, SOIC:SOIC-16_7.5x10.3mm_Pitch1.27mm, symbol IC_interface_i2c:TCA9534
- added U2: TCA9535, SSOP:TSSOP-24_4.4x7.8mm_Pitch0.65mm, symbol IC_interface_i2c:TCA9535
- C1, C10, C11, C12, C13, C14, C3, C4, C5, C6, C7, C8, C9: value 100nF -> C_0603
- CN1: footprint (none) -> pin_headers:Pin_Header_Straight_1x05
- CN2: footprint (none) -> connectors_JST_SH:Connectors_JST_SM04B-SRSS-TB
- CN3: renamed from P1; footprint (none) -> pin_headers:Pin_Header_Straight_1x04
- CN4: renamed from CN3; footprint (none) -> pin_headers:Pin_Header_Straight_1x04
- CN5: renamed from CN4; footprint (none) -> pin_headers:Pin_Header_Straight_1x04
- CN6: renamed from CN5; footprint (none) -> pin_headers:Pin_Header_Straight_1x04
- U1: value NE555 -> NE555-IC_logic; footprint (none) -> SOIC:SOIC-8_3.9x4.9mm_Pitch1.27mm; symbol SonarExtenderI2C-rescue:NE555-IC_logic -> IC_logic:NE555
- U10, U11, U12, U9: value 74xx590 -> 74xx590-IC_logic; footprint (none) -> SOIC:SOIC-16_3.9x9.9mm_Pitch1.27mm; symbol SonarExtenderI2C-rescue:74xx590-IC_logic -> IC_logic:74xx590
- U13: value 74xx4002 -> 74xx4002-IC_logic; footprint (none) -> SOIC:SOIC-14_3.9x8.7mm_Pitch1.27mm; symbol SonarExtenderI2C-rescue:74xx4002-IC_logic -> IC_logic:74xx4002
- U4: value 74xx138 -> 74xx138-IC_logic; footprint (none) -> SOIC:SOIC-16_3.9x9.9mm_Pitch1.27mm; symbol SonarExtenderI2C-rescue:74xx138-IC_logic -> IC_logic:74xx138
- U6: value 74xx175 -> 74xx175-IC_logic; footprint (none) -> SOIC:SOIC-16_3.9x9.9mm_Pitch1.27mm; symbol SonarExtenderI2C-rescue:74xx175-IC_logic -> IC_logic:74xx175
- U7: value 74xx04 -> 74xx04-IC_logic; footprint (none) -> SOIC:SOIC-14_3.9x8.7mm_Pitch1.27mm; symbol SonarExtenderI2C-rescue:74xx04-IC_logic -> IC_logic:74xx04
Connections:
- wire segments 326 -> 307
- no-connect marks 20 -> 19
Other:
- moved on the sheet: C3

Commit message: schematic changed
Parts:
- removed CN1: CONN_01X05, pin_headers:Pin_Header_Straight_1x05, symbol mechanical-connectors:CONN_01X05
- added MECH1, MECH2, MECH3, MECH4: MHP_3.2_5.0, MECH_mounting_holes:MHP_3.2_5.0, symbol MECH_mounting-holes:MHP_3.2_5.0
- added P1: CONN_01X06, Connector_PinHeader_2.54mm:PinHeader_1x06_P2.54mm_Horizontal, symbol mechanical-connectors:CONN_01X06
- CN3, CN4, CN5, CN6: footprint pin_headers:Pin_Header_Straight_1x04 -> Connector_PinHeader_2.54mm:PinHeader_1x04_P2.54mm_Horizontal
Connections:
- wire segments 307 -> 315
Changed lines of the file:
@@
 F 0 "CN3" H 10728 1041 50  0000 L CNN
 F 1 "CONN_01X04" H 10728 950 50  0000 L CNN
-F 2 "pin_headers:Pin_Header_Straight_1x04" H 10650 1000 50  0001 C CNN
+F 2 "Connector_PinHeader_2.54mm:PinHeader_1x04_P2.54mm_Horizontal" H 10650 1000 50  0001 C CNN
 F 3 "" H 10650 1000 50  0000 C CNN
 	1    10650 1000
@@
 F 0 "CN4" H 10728 1891 50  0000 L CNN
 F 1 "CONN_01X04" H 10728 1800 50  0000 L CNN
-F 2 "pin_headers:Pin_Header_Straight_1x04" H 10650 1850 50  0001 C CNN
+F 2 "Connector_PinHeader_2.54mm:PinHeader_1x04_P2.54mm_Horizontal" H 10650 1850 50  0001 C CNN
 F 3 "" H 10650 1850 50  0000 C CNN
 	1    10650 1850
@@
 F 0 "CN5" H 10728 2741 50  0000 L CNN
 F 1 "CONN_01X04" H 10728 2650 50  0000 L CNN
-F 2 "pin_headers:Pin_Header_Straight_1x04" H 10650 2700 50  0001 C CNN
+F 2 "Connector_PinHeader_2.54mm:PinHeader_1x04_P2.54mm_Horizontal" H 10650 2700 50  0001 C CNN
 F 3 "" H 10650 2700 50  0000 C CNN
 	1    10650 2700
@@
 F 0 "CN6" H 10728 3591 50  0000 L CNN
 F 1 "CONN_01X04" H 10728 3500 50  0000 L CNN
-F 2 "pin_headers:Pin_Header_Straight_1x04" H 10650 3550 50  0001 C CNN
+F 2 "Connector_PinHeader_2.54mm:PinHeader_1x04_P2.54mm_Horizontal" H 10650 3550 50  0001 C CNN
 F 3 "" H 10650 3550 50  0000 C CNN
 	1    10650 3550
@@
 T3
 $Comp
-L mechanical-connectors:CONN_01X05 CN1
-U 1 1 5EDEF79D
-P 800 3400
-F 0 "CN1" H 717 2975 50  0000 C CNN
-F 1 "CONN_01X05" H 717 3066 50  0000 C CNN
-F 2 "pin_headers:Pin_Header_Straight_1x05" H 717 3067 50  0001 C CNN
-F 3 "" H 800 3400 50  0000 C CNN
-	1    800  3400
-	-1   0    0    1
-$EndComp
-$Comp
 L power-supply:+3V3 #PWR04
 U 1 1 5EDF1594
-P 1250 3000
-F 0 "#PWR04" H 1250 2850 50  0001 C CNN
-F 1 "+3V3" V 1265 3128 50  0000 L CNN
-F 2 "" H 1250 3000 50  0000 C CNN
-F 3 "" H 1250 3000 50  0000 C CNN
-	1    1250 3000
+P 1350 3000
+F 0 "#PWR04" H 1350 2850 50  0001 C CNN
+F 1 "+3V3" V 1365 3128 50  0000 L CNN
+F 2 "" H 1350 3000 50  0000 C CNN
+F 3 "" H 1350 3000 50  0000 C CNN
+	1    1350 3000
 	1    0    0    -1
 $EndComp
@@
 	1000 3600 1100 3600
 Wire Wire Line
-	1000 3500 1250 3500
-Wire Wire Line
-	1250 3500 1250 3000
-Wire Wire Line
 	1000 3400 2100 3400
-Wire Wire Line
-	1500 3500 1500 3300
-Wire Wire Line
-	1500 3300 1000 3300
-Wire Wire Line
-	1500 3500 2100 3500
 Wire Wire Line
 	1800 3200 1000 3200
@@
 Wire Wire Line
 	1700 5000 2100 5000
+$Comp
+L MECH_mounting-holes:MHP_3.2_5.0 MECH1
+U 1 1 5EE2106C
+P 6000 2250
+F 0 "MECH1" H 6128 2296 50  0000 L CNN
+F 1 "MHP_3.2_5.0" H 6128 2205 50  0000 L CNN
+F 2 "MECH_mounting_holes:MHP_3.2_5.0" H 5900 2300 50  0001 C CNN
+F 3 "" H 6000 2250 50  0001 C CNN
+	1    6000 2250
+	0    -1   -1   0
+$EndComp
+$Comp
+L MECH_mounting-holes:MHP_3.2_5.0 MECH2
+U 1 1 5EE21BD3
+P 6250 2250
+F 0 "MECH2" H 6378 2296 50  0000 L CNN
+F 1 "MHP_3.2_5.0" H 6378 2205 50  0000 L CNN
+F 2 "MECH_mounting_holes:MHP_3.2_5.0" H 6150 2300 50  0001 C CNN
+F 3 "" H 6250 2250 50  0001 C CNN
+	1    6250 2250
+	0    -1   -1   0
+$EndComp
+$Comp
+L MECH_mounting-holes:MHP_3.2_5.0 MECH3
+U 1 1 5EE3E22C
+P 6500 2250
+F 0 "MECH3" H 6628 2296 50  0000 L CNN
+F 1 "MHP_3.2_5.0" H 6628 2205 50  0000 L CNN
+F 2 "MECH_mounting_holes:MHP_3.2_5.0" H 6400 2300 50  0001 C CNN
+F 3 "" H 6500 2250 50  0001 C CNN
+	1    6500 2250
+	0    -1   -1   0
+$EndComp
+$Comp
+L MECH_mounting-holes:MHP_3.2_5.0 MECH4
+U 1 1 5EE5AE63
+P 6750 2250
+F 0 "MECH4" H 6878 2296 50  0000 L CNN
+F 1 "MHP_3.2_5.0" H 6878 2205 50  0000 L CNN
+F 2 "MECH_mounting_holes:MHP_3.2_5.0" H 6650 2300 50  0001 C CNN
+F 3 "" H 6750 2250 50  0001 C CNN
+	1    6750 2250
+	0    -1   -1   0
+$EndComp
+Wire Wire Line
+	6750 2550 6750 2650
+Wire Wire Line
+	6750 2650 6500 2650
+Wire Wire Line
+	6000 2650 6000 2550
+Wire Wire Line
+	6250 2550 6250 2650
+Connection ~ 6250 2650
+Wire Wire Line
+	6250 2650 6000 2650
+Wire Wire Line
+	6500 2550 6500 2650
+Connection ~ 6500 2650
+Wire Wire Line
+	6500 2650 6250 2650
+Wire Wire Line
+	6250 2650 6250 2750
+$Comp
+L power-supply:GND #PWR0101
+U 1 1 5EF0B893
+P 6250 2750
+F 0 "#PWR0101" H 6250 2500 50  0001 C CNN
+F 1 "GND" H 6255 2577 50  0000 C CNN
+F 2 "" H 6250 2750 50  0000 C CNN
+F 3 "" H 6250 2750 50  0000 C CNN
+	1    6250 2750
+	1    0    0    -1
+$EndComp
+$Comp
+L mechanical-connectors:CONN_01X06 P1
+U 1 1 5EF1903E
+P 800 3350
+F 0 "P1" H 717 2785 50  0000 C CNN
+F 1 "CONN_01X06" H 717 2876 50  0000 C CNN
+F 2 "Connector_PinHeader_2.54mm:PinHeader_1x06_P2.54mm_Horizontal" H 717 2967 50  0000 C CNN
+F 3 "" H 800 3350 50  0000 C CNN
+	1    800  3350
+	-1   0    0    1
+$EndComp
+Wire Wire Line
+	1000 3500 2100 3500
+Wire Wire Line
+	1000 3300 1350 3300
+Wire Wire Line
+	1350 3300 1350 3000
+$Comp
+L power-supply:+5V #PWR0102
+U 1 1 5EF9110B
+P 1200 3000
+F 0 "#PWR0102" H 1200 2850 50  0001 C CNN
+F 1 "+5V" H 1215 3173 50  0000 C CNN
+F 2 "" H 1200 3000 50  0000 C CNN
+F 3 "" H 1200 3000 50  0000 C CNN
+	1    1200 3000
+	1    0    0    -1
+$EndComp
+Wire Wire Line
+	1000 3100 1200 3100
+Wire Wire Line
+	1200 3100 1200 3000
 $EndSCHEMATC

Commit message: finished pcb layout
Parts:
- added C2: C_0603, capacitors:C_0603, symbol devices:C_0603
- added L1: Label, labels:jecc_logo_7.2x2.2, symbol devices:Label
- added L2: Label, labels:Top, symbol devices:Label
- added L3: Label, labels:Bot, symbol devices:Label
- added L4: Label, labels:generationmake_logo, symbol devices:Label
- added R5, R6: 10k, resistors:R_0603, symbol devices:R_0603
Connections:
- wire segments 315 -> 333
- no-connect marks 19 -> 15
Other:
- moved on the sheet: U13
Changed lines of the file:
@@
 L IC_logic:74xx4002 U13
 U 1 1 5EF9FE5E
-P 10000 5550
-F 0 "U13" H 10000 6375 50  0000 C CNN
-F 1 "74xx4002-IC_logic" H 10000 6284 50  0000 C CNN
-F 2 "SOIC:SOIC-14_3.9x8.7mm_Pitch1.27mm" H 10000 5550 50  0001 C CNN
-F 3 "" H 10000 5550 50  0001 C CNN
-	1    10000 5550
-	1    0    0    -1
-$EndComp
-$Comp
-L power-supply:+3V3 #PWR047
-U 1 1 5EFA15D1
-P 10500 4850
-F 0 "#PWR047" H 10500 4700 50  0001 C CNN
-F 1 "+3V3" H 10515 5023 50  0000 C CNN
-F 2 "" H 10500 4850 50  0000 C CNN
-F 3 "" H 10500 4850 50  0000 C CNN
-	1    10500 4850
+P 10000 5650
+F 0 "U13" H 10000 6475 50  0000 C CNN
+F 1 "74xx4002-IC_logic" H 10000 6384 50  0000 C CNN
+F 2 "SOIC:SOIC-14_3.9x8.7mm_Pitch1.27mm" H 10000 5650 50  0001 C CNN
+F 3 "" H 10000 5650 50  0001 C CNN
+	1    10000 5650
 	1    0    0    -1
 $EndComp
@@
 $EndComp
 NoConn ~ 10300 5250
-NoConn ~ 9700 5400
-NoConn ~ 9700 5500
-NoConn ~ 9700 5600
-NoConn ~ 9700 5700
-Wire Wire Line
-	10300 5000 10500 5000
-Wire Wire Line
-	10500 5000 10500 4850
 Wire Wire Line
 	9700 5900 9600 5900
@@
 $EndComp
 Wire Wire Line
-	2500 2350 1750 2350
-Wire Wire Line
-	2500 2450 1750 2450
-Wire Wire Line
 	1750 2550 1850 2550
 Wire Wire Line
@@
 Wire Wire Line
 	1200 3100 1200 3000
+Wire Wire Line
+	2950 2350 2950 2250
+Wire Wire Line
+	1750 2350 2950 2350
+$Comp
+L devices:R_0603 R5
+U 1 1 5F074364
+P 2950 2150
+F 0 "R5" H 3009 2196 50  0000 L CNN
+F 1 "10k" H 3009 2105 50  0000 L CNN
+F 2 "resistors:R_0603" H 2950 2000 50  0001 C CNN
+F 3 "" H 2950 2150 50  0000 C CNN
+	1    2950 2150
+	1    0    0    -1
+$EndComp
+$Comp
+L devices:R_0603 R6
+U 1 1 5F07512E
+P 3200 2250
+F 0 "R6" H 3259 2296 50  0000 L CNN
+F 1 "10k" H 3259 2205 50  0000 L CNN
+F 2 "resistors:R_0603" H 3200 2100 50  0001 C CNN
+F 3 "" H 3200 2250 50  0000 C CNN
+	1    3200 2250
+	1    0    0    -1
+$EndComp
+Wire Wire Line
+	3200 2450 3200 2350
+Wire Wire Line
+	1750 2450 3200 2450
+Wire Wire Line
+	2950 2050 2950 2000
+Wire Wire Line
+	3200 2150 3200 2000
+Wire Wire Line
+	3200 2000 2950 2000
+Connection ~ 2950 2000
+Wire Wire Line
+	2950 2000 2950 1950
+$Comp
+L power-supply:+3V3 #PWR0103
+U 1 1 5F10D678
+P 2950 1950
+F 0 "#PWR0103" H 2950 1800 50  0001 C CNN
+F 1 "+3V3" H 2965 2123 50  0000 C CNN
+F 2 "" H 2950 1950 50  0000 C CNN
+F 3 "" H 2950 1950 50  0000 C CNN
+	1    2950 1950
+	1    0    0    -1
+$EndComp
+Wire Wire Line
+	9700 5450 9600 5450
+Wire Wire Line
+	9600 5450 9600 5550
+Connection ~ 9600 5900
+Wire Wire Line
+	9700 5750 9600 5750
+Connection ~ 9600 5750
+Wire Wire Line
+	9600 5750 9600 5900
+Wire Wire Line
+	9700 5650 9600 5650
+Connection ~ 9600 5650
+Wire Wire Line
+	9600 5650 9600 5750
+Wire Wire Line
+	9700 5550 9600 5550
+Connection ~ 9600 5550
+Wire Wire Line
+	9600 5550 9600 5650
+$Comp
+L power-supply:+3V3 #PWR0104
+U 1 1 5EEF0C5A
+P 10750 4400
+F 0 "#PWR0104" H 10750 4250 50  0001 C CNN
+F 1 "+3V3" H 10765 4573 50  0000 C CNN
+F 2 "" H 10750 4400 50  0000 C CNN
+F 3 "" H 10750 4400 50  0000 C CNN
+	1    10750 4400
+	1    0    0    -1
+$EndComp
+$Comp
+L devices:C_0603 C2
+U 1 1 5EEF0C60
+P 10750 4600
+F 0 "C2" H 10842 4646 50  0000 L CNN
+F 1 "C_0603" H 10842 4555 50  0000 L CNN
+F 2 "capacitors:C_0603" H 10750 4450 50  0001 C CNN
+F 3 "" H 10750 4600 50  0000 C CNN
+	1    10750 4600
+	1    0    0    -1
+$EndComp
+$Comp
+L power-supply:GND #PWR0105
+U 1 1 5EEF0C66
+P 10750 4750
+F 0 "#PWR0105" H 10750 4500 50  0001 C CNN
+F 1 "GND" H 10755 4577 50  0000 C CNN
+F 2 "" H 10750 4750 50  0000 C CNN
+F 3 "" H 10750 4750 50  0000 C CNN
+	1    10750 4750
+	1    0    0    -1
+$EndComp
+Wire Wire Line
+	10450 4450 10750 4450
+Wire Wire Line
+	10750 4450 10750 4400
+Wire Wire Line
+	10750 4450 10750 4500
+Connection ~ 10750 4450
+Wire Wire Line
+	10750 4700 10750 4750
+Wire Wire Line
+	10300 4950 10450 4950
+Wire Wire Line
+	10450 4950 10450 4450
+$Comp
+L devices:Label L1
+U 1 1 5EE35144
+P 1000 5500
+F 0 "L1" H 1228 5606 60  0000 L CNN
+F 1 "Label" H 1228 5500 60  0000 L CNN
+F 2 "labels:jecc_logo_7.2x2.2" H 1228 5394 60  0000 L CNN
+F 3 "" H 1000 5500 60  0000 C CNN
+	1    1000 5500
+	1    0    0    -1
+$EndComp
+$Comp
+L devices:Label L2
+U 1 1 5EE35975
+P 1000 5900
+F 0 "L2" H 1228 6006 60  0000 L CNN
+F 1 "Label" H 1228 5900 60  0000 L CNN
+F 2 "labels:Top" H 1228 5794 60  0000 L CNN
+F 3 "" H 1000 5900 60  0000 C CNN
+	1    1000 5900
+	1    0    0    -1
+$EndComp
+$Comp
+L devices:Label L3
+U 1 1 5EE55927
+P 1000 6300
+F 0 "L3" H 1228 6406 60  0000 L CNN
+F 1 "Label" H 1228 6300 60  0000 L CNN
+F 2 "labels:Bot" H 1228 6194 60  0000 L CNN
+F 3 "" H 1000 6300 60  0000 C CNN
+	1    1000 6300
+	1    0    0    -1
+$EndComp
+$Comp
+L devices:Label L4
+U 1 1 5EE75E1F
+P 2700 5500
+F 0 "L4" H 2928 5606 60  0000 L CNN
+F 1 "Label" H 2928 5500 60  0000 L CNN
+F 2 "labels:generationmake_logo" H 2928 5394 60  0000 L CNN
+F 3 "" H 2700 5500 60  0000 C CNN
+	1    2700 5500
+	1    0    0    -1
+$EndComp
 $EndSCHEMATC
