File: kicad_source/SonarExtenderI2C.sch (KiCad schematic (older format))
At the start: 44 parts, among them CN2 CONN_01X04, CN3 CONN_01X04, CN4 CONN_01X04, CN5 CONN_01X04, CN6 CONN_01X04, P1 CONN_01X06, U1 NE555-IC_logic, U10 74xx590-IC_logic, U11 74xx590-IC_logic, U12 74xx590-IC_logic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

Commit message: reacted to review
Parts:
- added C23, C24: 47uF 16V, capacitors:c_elec_6.3x4.5, symbol devices:CP_Small
- added D1, D2: Led_Small, LEDs:LED_0603, symbol devices:Led_Small
- added R7: 220, resistors:R_0603, symbol devices:R_0603
- added R8: 320, resistors:R_0603, symbol devices:R_0603
- C1: value C_0603 -> 1nF
- C10, C11, C12, C13, C14, C2, C3, C5, C6, C7, C8, C9: value C_0603 -> 100nF
- C4: value C_0603 -> 10nF
- R1: value R_0603 -> 120k
- R2: value R_0603 -> 12k
Connections:
- wire segments 333 -> 343
Changed lines of the file:
@@
 P 1700 4550
 F 0 "C3" H 1792 4596 50  0000 L CNN
-F 1 "C_0603" H 1792 4505 50  0000 L CNN
+F 1 "100nF" H 1792 4505 50  0000 L CNN
 F 2 "capacitors:C_0603" H 1700 4400 50  0001 C CNN
 F 3 "" H 1700 4550 50  0000 C CNN
@@
 P 7400 1900
 F 0 "C11" H 7492 1946 50  0000 L CNN
-F 1 "C_0603" H 7492 1855 50  0000 L CNN
+F 1 "100nF" H 7492 1855 50  0000 L CNN
 F 2 "capacitors:C_0603" H 7400 1750 50  0001 C CNN
 F 3 "" H 7400 1900 50  0000 C CNN
@@
 P 2750 1050
 F 0 "C5" H 2842 1096 50  0000 L CNN
-F 1 "C_0603" H 2842 1005 50  0000 L CNN
+F 1 "100nF" H 2842 1005 50  0000 L CNN
 F 2 "capacitors:C_0603" H 2750 900 50  0001 C CNN
 F 3 "" H 2750 1050 50  0000 C CNN
@@
 P 1200 1600
 F 0 "C1" H 1292 1646 50  0000 L CNN
-F 1 "C_0603" H 1292 1555 50  0000 L CNN
+F 1 "1nF" H 1292 1555 50  0000 L CNN
 F 2 "capacitors:C_0603" H 1200 1450 50  0001 C CNN
 F 3 "" H 1200 1600 50  0000 C CNN
@@
 P 1200 1300
 F 0 "R2" H 1259 1346 50  0000 L CNN
-F 1 "R_0603" H 1259 1255 50  0000 L CNN
+F 1 "12k" H 1259 1255 50  0000 L CNN
 F 2 "resistors:R_0603" H 1200 1150 50  0001 C CNN
 F 3 "" H 1200 1300 50  0000 C CNN
@@
 P 1200 950
 F 0 "R1" H 1259 996 50  0000 L CNN
-F 1 "R_0603" H 1259 905 50  0000 L CNN
+F 1 "120k" H 1259 905 50  0000 L CNN
 F 2 "resistors:R_0603" H 1200 800 50  0001 C CNN
 F 3 "" H 1200 950 50  0000 C CNN
@@
 P 2450 1850
 F 0 "C4" H 2542 1896 50  0000 L CNN
-F 1 "C_0603" H 2542 1805 50  0000 L CNN
+F 1 "10nF" H 2542 1805 50  0000 L CNN
 F 2 "capacitors:C_0603" H 2450 1700 50  0001 C CNN
 F 3 "" H 2450 1850 50  0000 C CNN
@@
 P 5050 900
 F 0 "C7" H 5142 946 50  0000 L CNN
-F 1 "C_0603" H 5142 855 50  0000 L CNN
+F 1 "100nF" H 5142 855 50  0000 L CNN
 F 2 "capacitors:C_0603" H 5050 750 50  0001 C CNN
 F 3 "" H 5050 900 50  0000 C CNN
@@
 P 5400 3350
 F 0 "C8" H 5492 3396 50  0000 L CNN
-F 1 "C_0603" H 5492 3305 50  0000 L CNN
+F 1 "100nF" H 5492 3305 50  0000 L CNN
 F 2 "capacitors:C_0603" H 5400 3200 50  0001 C CNN
 F 3 "" H 5400 3350 50  0000 C CNN
@@
 P 6500 3350
 F 0 "C10" H 6592 3396 50  0000 L CNN
-F 1 "C_0603" H 6592 3305 50  0000 L CNN
+F 1 "100nF" H 6592 3305 50  0000 L CNN
 F 2 "capacitors:C_0603" H 6500 3200 50  0001 C CNN
 F 3 "" H 6500 3350 50  0000 C CNN
@@
 	1    0    0    -1
 $EndComp
-$Comp
-L devices:C_0603 C12
-U 1 1 5EE4DE74
-P 7400 3400
-F 0 "C12" H 7492 3446 50  0000 L CNN
-F 1 "C_0603" H 7492 3355 50  0000 L CNN
-F 2 "capacitors:C_0603" H 7400 3250 50  0001 C CNN
-F 3 "" H 7400 3400 50  0000 C CNN
-	1    7400 3400
-	1    0    0    -1
-$EndComp
 Wire Wire Line
 	7850 3200 7400 3200
@@
 P 7400 5050
 F 0 "C13" H 7492 5096 50  0000 L CNN
-F 1 "C_0603" H 7492 5005 50  0000 L CNN
+F 1 "100nF" H 7492 5005 50  0000 L CNN
 F 2 "capacitors:C_0603" H 7400 4900 50  0001 C CNN
 F 3 "" H 7400 5050 50  0000 C CNN
@@
 P 7400 6550
 F 0 "C14" H 7492 6596 50  0000 L CNN
-F 1 "C_0603" H 7492 6505 50  0000 L CNN
+F 1 "100nF" H 7492 6505 50  0000 L CNN
 F 2 "capacitors:C_0603" H 7400 6400 50  0001 C CNN
 F 3 "" H 7400 6550 50  0000 C CNN
@@
 P 5850 5700
 F 0 "C9" H 5942 5746 50  0000 L CNN
-F 1 "C_0603" H 5942 5655 50  0000 L CNN
+F 1 "100nF" H 5942 5655 50  0000 L CNN
 F 2 "capacitors:C_0603" H 5850 5550 50  0001 C CNN
 F 3 "" H 5850 5700 50  0000 C CNN
@@
 P 3400 6250
 F 0 "C6" H 3492 6296 50  0000 L CNN
-F 1 "C_0603" H 3492 6205 50  0000 L CNN
+F 1 "100nF" H 3492 6205 50  0000 L CNN
 F 2 "capacitors:C_0603" H 3400 6100 50  0001 C CNN
 F 3 "" H 3400 6250 50  0000 C CNN
@@
 P 10750 4600
 F 0 "C2" H 10842 4646 50  0000 L CNN
-F 1 "C_0603" H 10842 4555 50  0000 L CNN
+F 1 "100nF" H 10842 4555 50  0000 L CNN
 F 2 "capacitors:C_0603" H 10750 4450 50  0001 C CNN
 F 3 "" H 10750 4600 50  0000 C CNN
@@
 	1    0    0    -1
 $EndComp
+$Comp
+L devices:R_0603 R7
+U 1 1 5EE5CCD4
+P 800 4200
+F 0 "R7" H 859 4246 50  0000 L CNN
+F 1 "220" H 859 4155 50  0000 L CNN
+F 2 "resistors:R_0603" H 800 4050 50  0001 C CNN
+F 3 "" H 800 4200 50  0000 C CNN
+	1    800  4200
+	1    0    0    -1
+$EndComp
+$Comp
+L devices:R_0603 R8
+U 1 1 5EE5D886
+P 1200 4200
+F 0 "R8" H 1259 4246 50  0000 L CNN
+F 1 "320" H 1259 4155 50  0000 L CNN
+F 2 "resistors:R_0603" H 1200 4050 50  0001 C CNN
+F 3 "" H 1200 4200 50  0000 C CNN
+	1    1200 4200
+	1    0    0    -1
+$EndComp
+$Comp
+L devices:Led_Small D1
+U 1 1 5EE5DBC0
+P 800 4450
+F 0 "D1" V 891 4382 50  0000 R CNN
+F 1 "Led_Small" V 800 4382 50  0000 R CNN
+F 2 "LEDs:LED_0603" V 709 4382 50  0000 R CNN
+F 3 "" V 800 4450 50  0000 C CNN
+	1    800  4450
+	0    -1   -1   0
+$EndComp
+$Comp
+L devices:Led_Small D2
+U 1 1 5EE5EA81
+P 1200 4450
+F 0 "D2" V 1291 4382 50  0000 R CNN
+F 1 "Led_Small" V 1200 4382 50  0000 R CNN
+F 2 "LEDs:LED_0603" V 1109 4382 50  0000 R CNN
+F 3 "" V 1200 4450 50  0000 C CNN
+	1    1200 4450
+	0    -1   -1   0
+$EndComp
+Wire Wire Line
+	800  4350 800  4300
+Wire Wire Line
+	1200 4350 1200 4300
+Wire Wire Line
+	800  4100 800  4050
+Wire Wire Line
+	1200 4100 1200 4050
+Wire Wire Line
+	800  4550 800  4600
+Wire Wire Line
+	1200 4550 1200 4600
+$Comp
+L power-supply:+3V3 #PWR0120
+U 1 1 5EF2589A
+P 800 4050
+F 0 "#PWR0120" H 800 3900 50  0001 C CNN
+F 1 "+3V3" H 815 4223 50  0000 C CNN
+F 2 "" H 800 4050 50  0000 C CNN
+F 3 "" H 800 4050 50  0000 C CNN
+	1    800  4050
+	1    0    0    -1
+$EndComp
+$Comp
+L power-supply:+5V #PWR0121
+U 1 1 5EF26456
+P 1200 4050
+F 0 "#PWR0121" H 1200 3900 50  0001 C CNN
+F 1 "+5V" H 1215 4223 50  0000 C CNN
+F 2 "" H 1200 4050 50  0000 C CNN
+F 3 "" H 1200 4050 50  0000 C CNN
+	1    1200 4050
+	1    0    0    -1
+$EndComp
+$Comp
+L power-supply:GND #PWR0122
+U 1 1 5EF26E6C
+P 800 4600
+F 0 "#PWR0122" H 800 4350 50  0001 C CNN
+F 1 "GND" H 805 4427 50  0000 C CNN
+F 2 "" H 800 4600 50  0000 C CNN
+F 3 "" H 800 4600 50  0000 C CNN
+	1    800  4600
+	1    0    0    -1
+$EndComp
+$Comp
+L power-supply:GND #PWR0123
+U 1 1 5EF27844
+P 1200 4600
+F 0 "#PWR0123" H 1200 4350 50  0001 C CNN
+F 1 "GND" H 1205 4427 50  0000 C CNN
+F 2 "" H 1200 4600 50  0000 C CNN
+F 3 "" H 1200 4600 50  0000 C CNN
+	1    1200 4600
+	1    0    0    -1
+$EndComp
+$Comp
+L devices:C_0603 C12
+U 1 1 5EE4DE74
+P 7400 3400
+F 0 "C12" H 7492 3446 50  0000 L CNN
+F 1 "100nF" H 7492 3355 50  0000 L CNN
+F 2 "capacitors:C_0603" H 7400 3250 50  0001 C CNN
+F 3 "" H 7400 3400 50  0000 C CNN
+	1    7400 3400
+	1    0    0    -1
+$EndComp
+$Comp
+L devices:CP_Small C24
+U 1 1 5EFA8459
+P 1250 7100
+F 0 "C24" H 1338 7191 50  0000 L CNN
+F 1 "47uF 16V" H 1338 7100 50  0000 L CNN
+F 2 "capacitors:c_elec_6.3x4.5" H 1338 7009 50  0000 L CNN
+F 3 "" H 1250 7100 50  0000 C CNN
+	1    1250 7100
+	1    0    0    -1
+$EndComp
+$Comp
+L devices:CP_Small C23
+U 1 1 5EFA9770
+P 700 7100
+F 0 "C23" H 788 7191 50  0000 L CNN
+F 1 "47uF 16V" H 788 7100 50  0000 L CNN
+F 2 "capacitors:c_elec_6.3x4.5" H 788 7009 50  0000 L CNN
+F 3 "" H 700 7100 50  0000 C CNN
+	1    700  7100
+	1    0    0    -1
+$EndComp
+Wire Wire Line
+	1250 7000 1250 6900
+Wire Wire Line
+	700  7000 700  6900
+Wire Wire Line
+	700  7200 700  7300
+Wire Wire Line
+	1250 7300 1250 7200
+$Comp
+L power-supply:GND #PWR0124
+U 1 1 5F051D79
+P 700 7300
+F 0 "#PWR0124" H 700 7050 50  0001 C CNN
+F 1 "GND" H 705 7127 50  0000 C CNN
+F 2 "" H 700 7300 50  0000 C CNN
+F 3 "" H 700 7300 50  0000 C CNN
+	1    700  7300
+	1    0    0    -1
+$EndComp
+$Comp
+L power-supply:GND #PWR0125
+U 1 1 5F0522F3
+P 1250 7300
+F 0 "#PWR0125" H 1250 7050 50  0001 C CNN
+F 1 "GND" H 1255 7127 50  0000 C CNN
+F 2 "" H 1250 7300 50  0000 C CNN
+F 3 "" H 1250 7300 50  0000 C CNN
+	1    1250 7300
+	1    0    0    -1
+$EndComp
+$Comp
+L power-supply:+3V3 #PWR0126
+U 1 1 5F074535
+P 700 6900
+F 0 "#PWR0126" H 700 6750 50  0001 C CNN
+F 1 "+3V3" H 715 7073 50  0000 C CNN
+F 2 "" H 700 6900 50  0000 C CNN
+F 3 "" H 700 6900 50  0000 C CNN
+	1    700  6900
+	1    0    0    -1
+$EndComp
+$Comp
+L power-supply:+5V #PWR0127
+U 1 1 5F07507E
+P 1250 6900
+F 0 "#PWR0127" H 1250 6750 50  0001 C CNN
+F 1 "+5V" H 1265 7073 50  0000 C CNN
+F 2 "" H 1250 6900 50  0000 C CNN
+F 3 "" H 1250 6900 50  0000 C CNN
+	1    1250 6900
+	1    0    0    -1
+$EndComp

Commit message: added led digikey order numbers
Parts:
- D1, D2: value Led_Small -> 150060GS75000

Commit message: added pause mode for automate
Parts:
- U1: symbol IC_logic:NE555 -> SonarExtenderI2C-rescue:NE555-IC_logic
- U10, U11, U12, U9: symbol IC_logic:74xx590 -> SonarExtenderI2C-rescue:74xx590-IC_logic
- U13: symbol IC_logic:74xx4002 -> SonarExtenderI2C-rescue:74xx4002-IC_logic
- U2: symbol IC_interface_i2c:TCA9535 -> SonarExtenderI2C-rescue:TCA9535-IC_interface_i2c
- U4: symbol IC_logic:74xx138 -> SonarExtenderI2C-rescue:74xx138-IC_logic
- U6: symbol IC_logic:74xx175 -> SonarExtenderI2C-rescue:74xx175-IC_logic
- U7: symbol IC_logic:74xx04 -> SonarExtenderI2C-rescue:74xx04-IC_logic
Connections:
- net labels added: PAUSE
- net labels removed: CNT0, CNT1, CNT2, CNT3
- wire segments 343 -> 344
- no-connect marks 15 -> 14
Changed lines of the file:
@@
 Wire Wire Line
 	2950 7000 3700 7000
-NoConn ~ 2950 7200
 NoConn ~ 2950 7300
 NoConn ~ 2950 7400
@@
 STATUS_ECHO
 Text GLabel 7300 1500 0    50   Input ~ 0
-CNT0
+ENABLE0
 Text GLabel 7300 3000 0    50   Input ~ 0
-CNT1
+ENABLE1
 Text GLabel 7300 4650 0    50   Input ~ 0
-CNT2
+ENABLE2
 Text GLabel 7300 6150 0    50   Input ~ 0
-CNT3
+ENABLE3
 Wire Wire Line
 	4300 3900 3850 3900
@@
 $EndComp
 $Comp
-L IC_logic:74xx590 U12
+L SonarExtenderI2C-rescue:74xx590-IC_logic U12
 U 1 1 5EE73281
 P 8200 6150
@@
 $EndComp
 $Comp
-L IC_logic:74xx590 U11
+L SonarExtenderI2C-rescue:74xx590-IC_logic U11
 U 1 1 5EE73231
 P 8200 4650
@@
 $EndComp
 $Comp
-L IC_logic:74xx590 U10
+L SonarExtenderI2C-rescue:74xx590-IC_logic U10
 U 1 1 5EE4DE46
 P 8200 3000
@@
 $EndComp
 $Comp
-L IC_logic:74xx590 U9
+L SonarExtenderI2C-rescue:74xx590-IC_logic U9
 U 1 1 5ED3FBEA
 P 8200 1500
@@
 $EndComp
 $Comp
-L IC_logic:74xx04 U7
+L SonarExtenderI2C-rescue:74xx04-IC_logic U7
 U 1 1 5EEE08C7
 P 5200 6400
@@
 $EndComp
 $Comp
-L IC_logic:74xx138 U4
+L SonarExtenderI2C-rescue:74xx138-IC_logic U4
 U 1 1 5F07A383
 P 2600 7050
@@
 $EndComp
 $Comp
-L IC_interface_i2c:TCA9535 U2
+L SonarExtenderI2C-rescue:TCA9535-IC_interface_i2c U2
 U 1 1 5F072FE1
 P 2600 4300
@@
 $EndComp
 $Comp
-L IC_logic:74xx175 U6
+L SonarExtenderI2C-rescue:74xx175-IC_logic U6
 U 1 1 5ED68086
 P 4650 4250
@@
 $EndComp
 $Comp
-L IC_logic:NE555 U1
+L SonarExtenderI2C-rescue:NE555-IC_logic U1
 U 1 1 5ED3F84C
 P 1950 1400
@@
 $EndComp
 $Comp
-L IC_logic:74xx4002 U13
+L SonarExtenderI2C-rescue:74xx4002-IC_logic U13
 U 1 1 5EF9FE5E
 P 10000 5650
@@
 	0    -1   -1   0
 $EndComp
+Wire Wire Line
+	2950 7200 3700 7200
+Text GLabel 3700 7200 2    50   Output ~ 0
+PAUSE
 $EndSCHEMATC
